File: minipci_module.sch (KiCad schematic (older format))
At the start: 3 parts, among them Con2 2041119-1

Commit message: Finalized project and generated all production files
Parts:
- added C1: 100n, Capacitors_Smd_0603:100nF_0603, symbol Capacitors_Smd0603:100n
- added C2: 10uF, Capacitors_Smd_0603:10uF_10V_0603, symbol Capacitors_Smd0603:10uF
Connections:
- net 3V3: now also C1.1, C2.1
- net GND: now also C1.2, C2.2
Changed lines of the file:
@@
 Wire Wire Line
 	6000 6000 5750 6000
+$Comp
+L Capacitors_Smd0603:100n C1
+U 1 1 600B8508
+P 7900 2150
+F 0 "C1" H 8031 2196 50  0000 L CNN
+F 1 "100n" H 8031 2105 50  0000 L CNN
+F 2 "Capacitors_Smd_0603:100nF_0603" H 7900 2150 60  0001 C CNN
+F 3 "Capacitors/Smd_0603/Components_Documentation/KEM_C1005_Y5V_SMD.pdf" H 7900 2150 60  0001 C CNN
+F 4 "SAMSUNG" H 7900 2150 50  0001 C CNN "Manufacturer"
+F 5 "CL10B104JB8NNNC" H 7900 2150 50  0001 C CNN "Manufacturer Part Number"
+F 6 "TME" H 7900 2150 50  0001 C CNN "Supplier"
+F 7 "CL10B104JB8NNNC" H 7900 2150 50  0001 C CNN "Supplier Part Number"
+F 8 "https://www.tme.eu/pl/details/cl10b104jb8nnnc/kondensatory-mlcc-smd-0603/samsung/" H 7900 2150 50  0001 C CNN "URL"
+F 9 "0,04540" H 7900 2150 50  0001 C CNN "Price@1pc"
+F 10 "0,02231" H 7900 2150 50  0001 C CNN "Price@1000pcs"
+F 11 "0603" H 7900 2150 50  0001 C CNN "Package"
+	1    7900 2150
+	1    0    0    -1
+$EndComp
+$Comp
+L Capacitors_Smd0603:10uF C2
+U 1 1 600B9083
+P 8400 2150
+F 0 "C2" H 8531 2196 50  0000 L CNN
+F 1 "10uF" H 8531 2105 50  0000 L CNN
+F 2 "Capacitors_Smd_0603:10uF_10V_0603" V 8250 2150 157 0001 C CNN
+F 3 "https://www.tme.eu/Document/08070be221b22b3ff38fe1f90e5753ee/C0603C106M9PACTU.pdf" V 8250 2150 157 0001 C CNN
+F 4 "KEMET" H 8400 2150 50  0001 C CNN "Manufacturer"
+F 5 "C0603C106M9PACTU" H 8400 2150 50  0001 C CNN "Manufacturer Part Number"
+F 6 "TME" H 8400 2150 50  0001 C CNN "Supplier"
+F 7 "C0603C106M9PAC" H 8400 2150 50  0001 C CNN "Supplier Part Number"
+F 8 "https://www.tme.eu/pl/details/c0603c106m9pac/kondensatory-mlcc-smd-0603/kemet/c0603c106m9pactu/" H 8400 2150 50  0001 C CNN "URL"
+F 9 "0,81309" H 8400 2150 50  0001 C CNN "Price@1pc"
+F 10 "0,20713" H 8400 2150 50  0001 C CNN "Price@1000pcs"
+F 11 "MW" H 8400 2150 50  0001 C CNN "Developer"
+F 12 "0603" H 8400 2150 50  0001 C CNN "Package"
+F 13 "C162265" H 8400 2150 50  0001 C CNN "LCSC Part # (optional)"
+	1    8400 2150
+	1    0    0    -1
+$EndComp
+$Comp
+L power:GND #PWR0108
+U 1 1 600BA36C
+P 7900 2450
+F 0 "#PWR0108" H 7900 2550 30  0001 C CNN
+F 1 "GND" H 7900 2350 30  0001 C CNN
+F 2 "" H 7900 2450 60  0000 C CNN
+F 3 "" H 7900 2450 60  0000 C CNN
+	1    7900 2450
+	1    0    0    -1
+$EndComp
+$Comp
+L power:GND #PWR0109
+U 1 1 600BAC88
+P 8400 2450
+F 0 "#PWR0109" H 8400 2550 30  0001 C CNN
+F 1 "GND" H 8400 2350 30  0001 C CNN
+F 2 "" H 8400 2450 60  0000 C CNN
+F 3 "" H 8400 2450 60  0000 C CNN
+	1    8400 2450
+	1    0    0    -1
+$EndComp
+$Comp
+L power:3V3_NO_GLOBAL #PWR27
+U 1 1 600BAFEE
+P 7900 1900
+F 0 "#PWR27" H 7900 2000 40  0001 C CNN
+F 1 "3V3" H 7850 2050 50  0000 L CNN
+F 2 "" H 7900 1900 60  0000 C CNN
+F 3 "" H 7900 1900 60  0000 C CNN
+	1    7900 1900
+	1    0    0    -1
+$EndComp
+$Comp
+L power:3V3_NO_GLOBAL #PWR28
+U 1 1 600BB47A
+P 8400 1900
+F 0 "#PWR28" H 8400 2000 40  0001 C CNN
+F 1 "3V3" H 8350 2050 50  0000 L CNN
+F 2 "" H 8400 1900 60  0000 C CNN
+F 3 "" H 8400 1900 60  0000 C CNN
+	1    8400 1900
+	1    0    0    -1
+$EndComp
+Wire Wire Line
+	8400 1900 8400 1950
+Wire Wire Line
+	8400 2350 8400 2450
+Wire Wire Line
+	7900 2450 7900 2350
+Wire Wire Line
+	7900 1950 7900 1900
 $EndSCHEMATC
