File: pi-hat-lorawan-gateway-minipci.sch (KiCad schematic (older format))
At the start: 1 part, among them Con1 RPi-Header-2x13

Commit message: Finalized project and generated all production files
Parts:
- added C3, C4: 10uF, Capacitors_Smd_0603:10uF_10V_0603, symbol Capacitors_Smd0603:10uF
- added D1: KPG-1608SURKC-T, Diodes:LED_KPG-1608SURKC-T, symbol Diodes:KPG-1608SURKC-T
- added R3: 200R, Resistor_Smd_0603:200R_0603, symbol Resistors_Smd0603:200R
- added U1: LD39200, Linear:LD39200PU33R, symbol Linear_Regulators:LD39200
Connections:
- net 3V3: now also Con1.17, R3.2
- net 5V: now also Con1.4, C3.1, U1.5 (EN), U1.6 (VIN)
- net GND: now also Con1.14, Con1.20, Con1.25, Con1.9, C3.2, C4.2, D1.2 (K), U1.3 (GND), U1.EP
- net GPIO17 renamed GPIO17(RTS)
- net GPIO18 renamed GPIO18(PWM)
- net RXD renamed GPIO15(RXD)
- net TXD renamed GPIO14(TXD)
- new net: D1.1 (A), R3.1
- new net MiniPci Express Module/POWER_IN_3V3: C4.1, U1.1 (VOUT), U1.2 (ADJ/SENSE)
- no-connect marks 6 -> 8
