File: pi-hat-lorawan-gateway-minipci.kicad_pcb (KiCad board)
At the start: 2 copper layers, 85 x 56 mm, 9 parts, among them Con1 RPi-Header-2x13, Con2 2041119-1, U1 LD39200

Commit message: Applied issue, regenerated gerbers
Connections:
- Con1 pad 1: 3V3 -> (no net)
- Con1 pad 16: /GPIO23 -> (no net)
- Con1 pad 17: 3V3 -> (no net)
- Con1 pad 3: /GPIO0(SDA) -> (no net)
- Con1 pad 5: /GPIO1(SCL) -> (no net)
- Con2 pad 17: (no net) -> GND
- Con2 pad 18: GND -> (no net)
- Con2 pad 19: /GPIO23 -> (no net)
- Con2 pad 20: GND -> (no net)
Routing:
- net /GPIO23: track 34.7 -> 0.00 mm
- net GND: track 9.49 -> 11.6 mm
