File: pi-hat-lorawan-gateway-minipci.kicad_sch (KiCad schematic)
At the start: 6 parts, among them Con1 RPi-Header-2x13, U1 LD39200

Commit message: Applied issue, regenerated gerbers
Connections:
- net MiniPci Express Module/POWER_IN_3V3 is gone; now on net 3V3: C4.1, U1.1 (VOUT), U1.2 (ADJ/SENSE)
- net 3V3: no longer Con1.1, Con1.17
- net GPIO23: no longer names the net of Con1.16
- no-connect marks 3 -> 7
